File: hope_project_digicam.kicad_sch (KiCad schematic)
At the start: 46 parts, among them J1 USB_C_Receptacle_USB2.0_16P, J2 SD_Card_Port, J3 Camera_Pin_Out, J4 Lipo batt in, J5 TFT_Pin_Socket, J6 extra, Q1 NMOS, Q2 PMOS, SW1 Cam Trigger, SW2 Reset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

Commit message: finished layout pretty much
Parts:
- removed TP10, TP11, TP12, TP7, TP8, TP9: TestPoint, TestPoint:TestPoint_Plated_Hole_D2.0mm, symbol Connector:TestPoint
- D2: footprint HOPE DigiCam:Shottky_Diode -> Diode_SMD:D_SOD-123
- J1: footprint HOPE DigiCam:USB_C_Receptacle -> Connector_USB:USB_C_Receptacle_GCT_USB4085
- SW1: footprint HOPE DigiCam:SW2_SW3 -> SWITCH_CAM:D6R_CNK
Connections:
- net CAM_D2: now also U1.8 (IO15); no longer U1.4 (IO4)
- net CAM_D3: now also U1.9 (IO16); no longer U1.5 (IO5)
- net CAM_D4: now also U1.10 (IO17); no longer U1.6 (IO6)
- net CAM_D5: now also U1.11 (IO18); no longer U1.7 (IO7)
- net CAM_D6: now also U1.12 (IO8); no longer U1.8 (IO15)
- net CAM_D7: now also U1.15 (IO3); no longer U1.9 (IO16)
- net CAM_D8: now also U1.16 (IO46); no longer U1.10 (IO17)
- net CAM_D9: now also U1.17 (IO9); no longer U1.11 (IO18)
- net CAM_HS: now also U1.20 (IO12); no longer U1.23 (IO21)
- net CAM_PC: now also U1.19 (IO11); no longer U1.12 (IO8)
- net CAM_SCL: now also U1.23 (IO21); no longer U1.39 (IO1)
- net CAM_SDA: now also U1.22 (IO14); no longer U1.38 (IO2)
- net CAM_TRIGGER: now also U1.39 (IO1); no longer U1.22 (IO14)
- net CAM_VS: now also U1.21 (IO13); no longer U1.24 (IO47)
- net CAM_XC: now also U1.18 (IO10); no longer U1.15 (IO3)
- net LED: now also U1.33 (IO40); no longer U1.26 (IO45)
- net SD_CS: now also U1.7 (IO7); no longer U1.18 (IO10)
- net SD_MISO: now also U1.4 (IO4); no longer U1.21 (IO13)
- net SD_MOSI: now also U1.6 (IO6); no longer U1.19 (IO11)
- net SD_SCK: now also U1.5 (IO5); no longer U1.20 (IO12)
- net TFT_CS: now also U1.31 (IO38); no longer U1.17 (IO9)
- net TFT_DC: now also U1.25 (IO48); no longer U1.16 (IO46)
- net TFT_LIT: now also U1.24 (IO47); no longer U1.25 (IO48)
- net TFT_SCK: now also U1.38 (IO2); no longer U1.31 (IO38)

Commit message: made silkscreen more readable
Parts:
- J6: footprint Connector_PinSocket_2.54mm:PinSocket_1x02_P2.54mm_Vertical -> Connector_PinHeader_2.54mm:PinHeader_1x02_P2.54mm_Vertical
Changed lines of the file:
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@@
 			)
 		)
-		(property "Footprint" "Connector_PinSocket_2.54mm:PinSocket_1x02_P2.54mm_Vertical"
+		(property "Footprint" "Connector_PinHeader_2.54mm:PinHeader_1x02_P2.54mm_Vertical"
 			(at 165.1 67.31 0)
 			(effects
